File: CAD/ssense-lte/ENV_SENSOR.kicad_sch (KiCad schematic)
At the start: 7 parts, among them Q2 Q_Photo_NPN, U4 SHTC3

Commit message: Backup commit
Parts:
- R35, R36: footprint Resistor_SMD:R_0603_1608Metric -> Resistor_SMD:R_0402_1005Metric
Changed lines of the file:
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@@
 			)
 		)
-		(property "Footprint" "Resistor_SMD:R_0603_1608Metric"
+		(property "Footprint" "Resistor_SMD:R_0402_1005Metric"
 			(at 128.27 85.09 0)
 			(effects
@@
 			)
 		)
-		(property "Footprint" "Resistor_SMD:R_0603_1608Metric"
+		(property "Footprint" "Resistor_SMD:R_0402_1005Metric"
 			(at 124.46 85.09 0)
 			(effects
