File: CAD/ssense-lte/POWER.kicad_sch (KiCad schematic)
At the start: 48 parts, among them J2 IEC61076-2_M8_A-coding_01x04_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, SW3 KMR223NGLFG, U1 LV2862XDDC, U3 nPM1300-QEXX, U6 THVD1450DR

Commit message: Backup commit
Parts:
- BT1: value BH-18650-PC2 -> Keystone 1042; footprint Methanesense:BatteryHolder_MPD_BH-18650-PC2 -> Battery:BatteryHolder_Keystone_1042_1x18650
- R1, R10, R11, R13, R14, R15, R16, R3, R4, R7, R8, R9: footprint Resistor_SMD:R_0603_1608Metric -> Resistor_SMD:R_0402_1005Metric
Connections:
- net A_P: now also R11.2, R12.1; no longer R10.2, R12.2
- net B_N: now also R10.2, R12.2; no longer R11.2, R12.1
Changed lines of the file:
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@@
 	(wire
 		(pts
-			(xy 87.63 46.99) (xy 87.63 49.53)
+			(xy 44.45 71.12) (xy 43.18 71.12)
 		)
 		(stroke
@@
 	(wire
 		(pts
-			(xy 113.03 54.61) (xy 120.65 54.61)
+			(xy 87.63 46.99) (xy 87.63 49.53)
 		)
 		(stroke
@@
 	(wire
 		(pts
-			(xy 41.91 54.61) (xy 41.91 101.6)
+			(xy 113.03 54.61) (xy 120.65 54.61)
 		)
 		(stroke
@@
 	(wire
 		(pts
+			(xy 43.18 71.12) (xy 43.18 73.66)
+		)
+		(stroke
+			(width 0)
+			(type default)
+		)
+	)
+	(wire
+		(pts
 			(xy 165.1 127) (xy 171.45 127)
 		)
@@
 	(wire
 		(pts
+			(xy 44.45 72.39) (xy 44.45 93.98)
+		)
+		(stroke
+			(width 0)
+			(type default)
+		)
+	)
+	(wire
+		(pts
 			(xy 219.71 48.26) (xy 214.63 48.26)
 		)
@@
 		)
 	)
+	(wire
+		(pts
+			(xy 41.91 73.66) (xy 41.91 101.6)
+		)
+		(stroke
+			(width 0)
+			(type default)
+		)
+	)
 	(polyline
 		(pts
@@
 	(wire
 		(pts
+			(xy 44.45 52.07) (xy 44.45 71.12)
+		)
+		(stroke
+			(width 0)
+			(type default)
+		)
+	)
+	(wire
+		(pts
 			(xy 44.45 175.26) (xy 44.45 173.99)
 		)
@@
 	(wire
 		(pts
-			(xy 44.45 52.07) (xy 44.45 93.98)
+			(xy 43.18 73.66) (xy 41.91 73.66)
 		)
 		(stroke
@@
 	(wire
 		(pts
+			(xy 41.91 54.61) (xy 41.91 72.39)
+		)
+		(stroke
+			(width 0)
+			(type default)
+		)
+	)
+	(wire
+		(pts
 			(xy 92.71 114.3) (xy 99.06 114.3)
 		)
@@
 	(wire
 		(pts
+			(xy 41.91 72.39) (xy 44.45 72.39)
+		)
+		(stroke
+			(width 0)
+			(type default)
+		)
+	)
+	(wire
+		(pts
 			(xy 255.27 116.84) (xy 252.73 116.84)
 		)
@@
 	)
 	(label "B_N"
-		(at 49.53 101.6 180)
+		(at 41.91 54.61 180)
 		(effects
 			(font
@@
 	)
 	(label "A_P"
-		(at 49.53 93.98 180)
+		(at 41.91 52.07 180)
 		(effects
 			(font
@@
 			)
 		)
-		(property "Footprint" "Resistor_SMD:R_0603_1608Metric"
+		(property "Footprint" "Resistor_SMD:R_0402_1005Metric"
 			(at 161.29 117.602 90)
 			(effects
@@
 			)
 		)
-		(property "Footprint" "Resistor_SMD:R_0603_1608Metric"
+		(property "Footprint" "Resistor_SMD:R_0402_1005Metric"
 			(at 104.902 64.77 90)
 			(effects
@@
 			)
 		)
-		(property "Footprint" "Resistor_SMD:R_0603_1608Metric"
+		(property "Footprint" "Resistor_SMD:R_0402_1005Metric"
 			(at 102.362 105.41 90)
 			(effects
@@
 			)
 		)
-		(property "Footprint" "Resistor_SMD:R_0603_1608Metric"
+		(property "Footprint" "Resistor_SMD:R_0402_1005Metric"
 			(at 104.902 73.66 90)
 			(effects
@@
 			)
 		)
-		(property "Footprint" "Resistor_SMD:R_0603_1608Metric"
+		(property "Footprint" "Resistor_SMD:R_0402_1005Metric"
 			(at 110.49 99.568 90)
 			(effects
@@
 			)
 		)
-		(property "Footprint" "Resistor_SMD:R_0603_1608Metric"
+		(property "Footprint" "Resistor_SMD:R_0402_1005Metric"
 			(at 132.842 71.12 90)
 			(effects
@@
 			)
 		)
-		(property "Footprint" "Resistor_SMD:R_0603_1608Metric"
+		(property "Footprint" "Resistor_SMD:R_0402_1005Metric"
 			(at 110.49 116.078 90)
 			(effects
@@
 			)
 		)
-		(property "Footprint" "Resistor_SMD:R_0603_1608Metric"
+		(property "Footprint" "Resistor_SMD:R_0402_1005Metric"
 			(at 132.842 62.23 90)
 			(effects
@@
 			)
 		)
-		(property "Footprint" "Resistor_SMD:R_0603_1608Metric"
+		(property "Footprint" "Resistor_SMD:R_0402_1005Metric"
 			(at 59.69 102.108 90)
 			(effects
@@
 			)
 		)
-		(property "Footprint" "Resistor_SMD:R_0603_1608Metric"
+		(property "Footprint" "Resistor_SMD:R_0402_1005Metric"
 			(at 59.69 97.028 90)
 			(effects
@@
 			)
 		)
-		(property "Value" "BH-18650-PC2"
+		(property "Value" "Keystone 1042"
 			(at 48.26 170.8784 0)
 			(effects
@@
 			)
 		)
-		(property "Footprint" "Methanesense:BatteryHolder_MPD_BH-18650-PC2"
+		(property "Footprint" "Battery:BatteryHolder_Keystone_1042_1x18650"
 			(at 44.45 169.926 90)
 			(effects
@@
 			)
 		)
-		(property "Footprint" "Resistor_SMD:R_0603_1608Metric"
+		(property "Footprint" "Resistor_SMD:R_0402_1005Metric"
 			(at 110.49 103.378 90)
 			(effects
@@
 			)
 		)
-		(property "Footprint" "Resistor_SMD:R_0603_1608Metric"
+		(property "Footprint" "Resistor_SMD:R_0402_1005Metric"
 			(at 97.282 110.49 90)
 			(effects
