File: CAD/ssense-lte/ssense-lte.kicad_pcb (KiCad board)
At the start: 4 copper layers, 96.5 x 36 mm, 130 parts, among them J1 HIROSE ELECTRIC U.FL-R-SMT-1, J2 IEC61076-2_M8_A-coding_01x04_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, J3 693043020611, J4 HIROSE ELECTRIC U.FL-R-SMT-1, J6 JLINK, Q3 IRLML6401, Q4 MMBT3906, SW1 KMR223NGLFG, SW3 KMR223NGLFG, U1 LV2862XDDC, U3 nPM1300-QEXX, U4 SHTC3, U5 nRF9160-SICA, U6 THVD1450DR, U8 USBLC6-4SC6, U9 TPS22917DBV, X1 KC3225K75.0000C1GE00

Commit message: Backup commit
Parts:
- removed kibuzzard-680B71B4: G***, kibuzzard-680B71B4
- removed kibuzzard-680B72A0: G***, kibuzzard-680B72A0
- removed kibuzzard-680B72CB: G***, kibuzzard-680B72CB
- removed kibuzzard-680B72EC: G***, kibuzzard-680B72EC
- removed kibuzzard-680B7325: G***, kibuzzard-680B7325
- removed kibuzzard-680B73BF: G***, kibuzzard-680B73BF
- removed kibuzzard-680B73D9: G***, kibuzzard-680B73D9
- BT1: value BH-18650-PC2 -> Keystone 1042; footprint Methanesense:BatteryHolder_MPD_BH-18650-PC2 -> Battery:BatteryHolder_Keystone_1042_1x18650
- R1, R10, R11, R13, R14, R15, R16, R17, R18, R19, R20, R29, R3, R35, R36, R38, R39, R4, R40, R41, R42, R43, R44, R45, R7, R8, R9: footprint Resistor_SMD:R_0603_1608Metric -> Resistor_SMD:R_0402_1005Metric
- moved TP15 113.8 mm to (180.8, 86.5)
- moved TP4 105.4 mm to (180.8, 83.5)
- moved TP3 101.6 mm to (180.8, 80.4)
- moved TP2 100.5 mm to (180.8, 77.4)
- moved TP1 98.3 mm to (180.8, 74.3)
- moved TP16 74.1 mm to (180.8, 69.3)
- moved kibuzzard-689F1011 58.0 mm to (133.5, 90.5)
- moved F1 57.9 mm to (113.5, 68.0), turned to 90 degrees
- moved BT1 37.5 mm to (91.4, 71.8), turned to 180 degrees
- moved D12 34.1 mm to (86.5, 75.5)
- moved C99 25.5 mm to (98.0, 75.5), turned to 0 degrees
- moved R40 25.2 mm to (91.1, 78.2), turned to -90 degrees
- moved C3 25.1 mm to (94.4, 80.6)
- moved X1 25.1 mm to (93.8, 78.0)
- moved Q3 24.4 mm to (90.6, 80.9)
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Connections:
- R10 pad 2: /POWER/A_P -> /POWER/B_N
- R11 pad 2: /POWER/B_N -> /POWER/A_P
- R12 pad 1: /POWER/B_N -> /POWER/A_P
- R12 pad 2: /POWER/A_P -> /POWER/B_N
Routing:
- net ~{RESET}: track 0.00 -> 24.4 mm, vias 0 -> 2
- net SWDCLK: track 0.00 -> 20.3 mm
- net SWDIO: track 0.00 -> 18.8 mm, vias 0 -> 2
- net Net-(J3-RST): track 0.00 -> 15.2 mm
- net /POWER/A_P: track 0.00 -> 14.7 mm
- net /POWER/B_N: track 0.00 -> 13.9 mm
- net GND: track 217.7 -> 205.6 mm, vias 167 -> 149
- net P0.04: track 0.85 -> 10.9 mm, vias 1 -> 2
- net /POWER/VIN: track 0.00 -> 7.96 mm
- net VCC: track 44.5 -> 36.6 mm, vias 10 -> 8
- net Net-(J3-CLK): track 2.42 -> 10.2 mm
- net Net-(Q3-D): track 0.00 -> 5.78 mm
- net Net-(D12-K): track 0.00 -> 4.71 mm
- net COEX0: track 0.00 -> 4.35 mm
- net P0.06: track 0.00 -> 3.95 mm
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- removed copper zone on In2.Cu, net +BATT
Other:
- board size 96.5 x 36 mm -> 113 x 25.1 mm
